File: _saved_atxmega_playground.sch (KiCad schematic (older format))
At the start: 119 parts, among them CON1 AVR-PDI-6, IC1 ATXMEGA32A4U-A, P1 USB_OTG, P2 CONN_01X02, P3 CONN_01X02, P4 CONN_01X06, P5 CONN_01X03, P6 CONN_01X04, P7 CONN_01X04, P8 CONN_01X07, Q1 PMOS, Q2 NMOS, Q3 NMOS, Q4 NMOS, U1 NCP346, U10 WS2812B, U11 WS2812B, U12 74HC595_F, U13 74HC595_F, U14 AT25SF041, U15 REF195, U16 AD7708, U17 MPXH6101A, U18 LM35, U2 LM3940, U3 ADM3315E, U4 HI-3110, U5 INA139, U6 WS2812B, U7 SN65220, U8 WS2812B, U9 PI4ULS5V201, Y1 16MHz, Y2 32.768kHz

Commit message: Basic layout, component positions mostly final
Parts:
- added TP4, TP5: TEST, atxmega:TESTPOINT, symbol TEST
- TP3: footprint (none) -> atxmega:TESTPOINT
Connections:
- wire segments 489 -> 494
