File: atxmega_playground.kicad_pcb (KiCad board)
At the start: 2 copper layers, 67.6 x 63.5 mm, 122 parts, among them CON1 AVR-PDI-6, IC1 ATXMEGA32A4U-A, P1 USB_OTG, P2 CONN_01X05, P3 CONN_01X02, P5 CONN_01X03, P7 CONN_01X04, Q1 PMOS, Q2 NMOS, Q3 NMOS, Q4 NMOS, U1 NCP346, U10 WS2812B, U11 WS2812B, U12 74HC595_F, U13 74HC595_F, U14 AT25SF041, U15 REF195, U16 AD7708, U17 MPXH6101A, U18 LM35, U2 LM3940, U3 ADM3315E, U4 HI-3110, U5 INA139, U6 WS2812B, U7 SN65220, U8 WS2812B, U9 PI4ULS5V201, Y1 16MHz, Y2 32.768kHz

Commit message: Final touches
Other:
- board text added: "+12V"
- board text added: "+5V"
- board text added: "GND"
- board text added: "RX"
- board text added: "TX"
- board text added: "Version 1.0"
- board text added: "XMega Playground"
- board text removed: "USB (mm) Clearance: 0.195072 Width: 0.184302"
Changed lines of the file:
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@@
     (area 79.172999 26.340999 146.887001 89.991001)
     (thickness 1.6)
-    (drawings 5)
+    (drawings 11)
     (tracks 1194)
     (zones 0)
@@
     (tags "capacitor 0805")
     (attr smd)
-    (fp_text reference C15 (at 3.2258 -0.0254 450) (layer F.SilkS)
+    (fp_text reference C15 (at -3.3528 0.0508 450) (layer F.SilkS)
       (effects (font (size 1 1) (thickness 0.15)))
     )
@@
     (tags "capacitor 0805")
     (attr smd)
-    (fp_text reference C16 (at 3.2766 0.254 270) (layer F.SilkS)
+    (fp_text reference C16 (at -3.4798 0.1016 270) (layer F.SilkS)
       (effects (font (size 1 1) (thickness 0.15)))
     )
@@
     (tags "SOIC 1.27")
     (attr smd)
-    (fp_text reference U18 (at 1.524 -3.7338) (layer F.SilkS)
+    (fp_text reference U18 (at 1.524 -3.4036) (layer F.SilkS)
       (effects (font (size 1 1) (thickness 0.15)))
     )
@@
     (tags SOT-23-6)
     (attr smd)
-    (fp_text reference U9 (at 0.8636 -2.1336) (layer F.SilkS)
+    (fp_text reference U9 (at 2.921 0.7874) (layer F.SilkS)
       (effects (font (size 1 1) (thickness 0.15)))
     )
@@
     )
   )
-  (gr_text "USB (mm)\nClearance: 0.195072\nWidth: 0.184302" (at 171.831 41.0718) (layer F.SilkS)
+  (gr_text TX (at 98.7044 63.3476) (layer F.SilkS)
+    (effects (font (size 1 1) (thickness 0.25)))
+  )
+  (gr_text RX (at 98.8568 66.7512) (layer F.SilkS)
+    (effects (font (size 1 1) (thickness 0.25)))
+  )
+  (gr_text +12V (at 134.9502 67.818 360) (layer F.SilkS)
+    (effects (font (size 1 1) (thickness 0.25)))
+  )
+  (gr_text GND (at 129.9718 74.803) (layer F.SilkS)
+    (effects (font (size 1 1) (thickness 0.25)))
+  )
+  (gr_text +5V (at 129.794 77.9526) (layer F.SilkS)
+    (effects (font (size 1 1) (thickness 0.25)))
+  )
+  (gr_text "Version 1.0" (at 101.9048 29.8196) (layer F.SilkS)
+    (effects (font (size 1 1) (thickness 0.25)))
+  )
+  (gr_text "XMega Playground" (at 106.934 27.6606) (layer F.SilkS)
     (effects (font (size 1.5 1.5) (thickness 0.3)))
   )

Commit message: First revision, finalized!
Parts:
- added C10: 33uF, atxmega:R_1206, B.Cu at (142.0, 75.1)
- added C17: 1uF, atxmega:R_1206, F.Cu at (110.5, 74.9)
- added G***: LOGO, atxmega:cuauv_prop_small, B.Cu at (142.4, 30.4)
Connections:
- IC1 pad 7: (no net) -> /CAN_INT
- U14 pad 3: (no net) -> +3V3
- U14 pad 7: (no net) -> +3V3
- U4 pad 18: (no net) -> /CAN_INT
Routing:
- net /CAN_INT: track 0.00 -> 28.7 mm, vias 0 -> 2
- net +3V3: track 298.8 -> 325.9 mm, vias 21 -> 24
- net GND: track 148.1 -> 154.0 mm
- net Net-(C17-Pad1): track 16.0 -> 19.1 mm
